File: hardware/kicad/ESP32.kicad_sch (KiCad schematic)
At the start: 4 parts, among them J1 Conn_01x02, U1 XIAO-ESP32-C6

Commit message: chore: added licensing
Other:
- title: (none) -> Air Quality Monitor
Changed lines of the file:
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@@
 	(generator_version "9.0")
 	(paper "A4")
+	(title_block
+		(title "Air Quality Monitor")
+		(date "2026-05-10")
+		(rev "v1.0")
+		(comment 1 "Author: Alejandro Macias Chaves")
+		(comment 2 "Licensed under CERN-OHL-P-2.0")
+	)
 	(text "Anotaciones:\n- Por la etiqueta \"SDAX\" el MCU envia datos a la pantalla\n- Por la etiqueta \"SDOX\" el MCU recive datos de la pantalla\n- La etiqueta DCX de la pantalla se corresponde al Serial Clock cuando esta esta configurada para SPI\n- La etiqueta WRX de la pantalla se corresponde con el Data/Command selection de la pantalla cuando esta esta configurada en 4-wire SPI"
 		(exclude_from_sim no)
