File: hardware/kicad/air_quality_pcb.kicad_pcb (KiCad board)
At the start: 2 copper layers, 75 x 75 mm, 29 parts, among them IC1 SCD41-D-R2, IC2 SGP41-D-R4, IC3 TPS61027DRCR, J1 Conn_01x02, J2 52435-2871, U1 XIAO-ESP32-C6, U2 MQ-6, U3 MQ-6

Commit message: chore: added licensing
Parts:
- added REF**: OSHW-Logo2_9.8x8mm_SilkScreen, Symbol:OSHW-Logo2_9.8x8mm_SilkScreen, F.Cu at (108.4, 61.9)
Other:
- board text added: "Licensed under CERN-OHL-P v2.0"
