File: hardware/kicad/air_quality_pcb.kicad_sch (KiCad schematic)
At the start: 0 parts

Commit message: chore: added licensing
Other:
- title: Air Quality Monitoring Device -> Air Quality Monitor
Changed lines of the file:
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@@
 	(paper "A4")
 	(title_block
-		(title "Air Quality Monitoring Device")
+		(title "Air Quality Monitor")
+		(date "2026-05-10")
+		(rev "v1.0")
+		(comment 1 "Author: Alejandro Macias Chaves")
+		(comment 2 "Licensed under CERN-OHL-P-2.0")
 	)
 	(sheet
