File: hardware/kicad/sensors.kicad_sch (KiCad schematic)
At the start: 25 parts, among them IC1 SCD41-D-R2, IC2 SGP41-D-R4, IC3 TPS61027DRCR, J2 52435-2871, U2 MQ-6, U3 MQ-6

Commit message: chore: added licensing
Other:
- title: (none) -> Air Quality Monitor
Changed lines of the file:
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@@
 	(generator_version "9.0")
 	(paper "A3")
+	(title_block
+		(title "Air Quality Monitor")
+		(date "2026-05-10")
+		(rev "v1.0")
+		(comment 1 "Author: Alejandro Macias Chaves")
+		(comment 2 "Licensed under CERN-OHL-P-2.0")
+	)
 	(rectangle
 		(start 154.94 39.37)
